File: ac-adapter.brd (EAGLE design)
At the start: 81.3 x 73.7 mm, 45 parts, among them IC2 TL431, Q1 300V5A, Q2 300V5A, Q3 TLP621-1, T1 COMMON_FILTER-SU10VFC, T2 TRANSFORMAER_FLYBACK-PQ2620, T3 COMMON_FILTER-SMALL

Commit message: 定数決まらん
Parts:
- removed T3: COMMON_FILTER-SMALL, my_rcl:COMMON_FILTER__SMALL
- added C10, C3: 100p, my_rcl:1608
- added C11: 10000p, my_rcl:1608
- added C4, R3, R9: (no value), my_rcl:1608
- added C5, C7: 0.1u, my_rcl:1608
- added C6: 1kV 470p, my_rcl:C050
- added C8: 100u, my_rcl:E2.5-6.5
- added C9: 1000p, my_rcl:1608
- added D2: 100V0.1A, my_rcl:SOD123
- added D3: 600V1A, my_rcl:D0204/7
- added D6: 12V, my_rcl:SOD123
- added IC1: NCP13992, my_ic:SO16-NCP13992
- added Q4: BSS128, my_ic:SC59
- added R11, R4: 10, my_rcl:1608
- added R12: 1.5k, my_rcl:1608
- added R5: 1M, my_rcl:0204/7
- added R6, R7: 10k, my_rcl:1608
- added R8: 47k, my_rcl:1608
- C17, C18: value 1000u -> 470u
- C2: device my_rcl:E5-16A -> my_rcl:E5-16A2
- C24: value 0.1u -> 3300p
- Q1, Q2: value 300V5A -> 300V 5A
- R1, R2: value 22 -> 10; device my_rcl:0204/7 -> my_rcl:2012
- R10, R13: value 22 -> 10; device my_rcl:0207/2V -> my_rcl:2012
- R17: value 1.5k -> 5k
- moved L3 83.3 mm to (52.2, 52.1)
- moved C15 37.7 mm to (52.1, 8.26)
- moved F1 21.9 mm to (32.4, 51.4)
- moved D1 21.8 mm to (6.35, 33.7)
- moved TP1 19.7 mm to (36.2, 62.9)
- moved TP2 19.1 mm to (29.2, 62.9)
- moved C23 17.3 mm to (34.3, 32.4), turned to 90 degrees
- moved R15 16.4 mm to (71.1, 3.49)
- moved R13 16.2 mm to (84.8, 14.9), flipped to the bottom, turned to 90 degrees
- moved IC2 16.2 mm to (66.5, 5.08)
- moved Q1 16.1 mm to (29.8, 40.6), turned to 0 degrees
- moved C24 16.0 mm to (64.3, 3.97)
- moved R14 15.8 mm to (68.9, 3.49)
- moved R19 15.0 mm to (61.9, 3.97)
- moved Q3 14.2 mm to (52.4, 3.17)
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Connections:
- removed net N$30: T3.1, TP2.1
- removed net N$31: F1.2, T3.4
- removed net N$43: Q3.3
- removed net N$44: C2.-, C23.2, D1.4, Q2.3, R21.1
- new net N$12: IC1.8, R7.2
- new net N$13: C3.1, D6.1, IC1.7, R8.2
- new net N$14: C4.1, C6.2, IC1.6, R9.2
- new net N$15: IC1.4, R6.2
- new net N$16: IC1.14, R1.1
- new net N$17: IC1.12, R2.2
- new net N$18: C5.1, D3.2, IC1.16
- new net N$19: IC1.3, Q4.2, R3.2
- new net N$20: C10.1, IC1.5, Q3.4
- new net N$21: Q4.3, R5.1
- new net N$23: C11.1, R12.2
- new net N$24: C9.1, D2.1, R4.1
- new net N$25: D3.1, R11.2
- new net PFC_MODE: IC1.9, Q4.1
- new net PGND: C10.2, C15.2, C2.-, C23.2, C3.2, C4.2, C7.2, C8.-, C9.2, D1.4, IC1.11, Q2.3, Q3.3, R21.1, R3.1, R6.1, R7.1, R8.1, R9.1, T2.5
- new net VCC: C7.1, C8.+, D2.2, D6.2, IC1.10, R11.1
- net N$1: now also F1.2; no longer T3.3
- net N$11: no longer L3.4, L3.5
- net N$2: now also R1.2; no longer R1.1
- net N$22: now also R4.2, T2.6; no longer Q3.4
- net N$26: now also TP2.1; no longer T3.2
- net N$3: now also R13.1; no longer R13.2
- net N$34: now also R12.1
- net N$35: now also R13.2; no longer C19.2
- net N$40: now also C11.2, C19.2; no longer R13.1
- net N$8: now also C6.1
- net SW: now also C5.2, IC1.15, L3.4; no longer L3.1, L3.2, L3.3
- net VH: now also IC1.1, R5.2
Routing:
- net PGND: track 0.00 -> 83.1 mm, vias 0 -> 51
- net SW: track 0.00 -> 55.3 mm
- net VH: track 0.00 -> 51.1 mm
- net VCC: track 0.00 -> 43.0 mm, vias 0 -> 1
- net N$20: track 0.00 -> 36.4 mm
- net N$5: track 0.00 -> 28.8 mm
- net N$40: track 0.00 -> 27.7 mm
- net N$19: track 0.00 -> 22.4 mm
- net N$14: track 0.00 -> 21.2 mm, vias 0 -> 1
- net N$4: track 0.00 -> 20.5 mm
- net GND: track 0.00 -> 20.1 mm, vias 0 -> 10
- net N$1: track 0.00 -> 17.6 mm
- net N$26: track 0.00 -> 14.1 mm
- net N$34: track 0.00 -> 12.8 mm, vias 0 -> 1
- net N$2: track 0.00 -> 11.9 mm
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- added copper zone on layer 1, net GND
- added copper zone on layer 16, net GND
- added copper zone on layer 16, net N$35
- added copper zone on layer 16, net N$36
- added copper zone on layer 1, net N$40
- added copper zone on layer 16, net N$7
- added copper zone on layer 1, net PGND
- added copper zone on layer 16, net PGND
- added copper zone on layer 16, net V+
- added copper zone on layer 16, net V-
Other:
- board size 81.3 x 73.7 mm -> 87.6 x 73 mm
- board text added: "LLC Power Supply v2"
- board text removed: "LLC AC adapter ±20V 3A"

Commit message: 微修正
Parts:
- C4: value (none) -> 100p
- C6: value 1kV 470p -> 1kV 22p
- R17: value 5k -> 10k
- R18: value 1.5k -> 10k
- R3: value (none) -> 10k
- R9: value (none) -> 330
Connections:
- net N$29: now also R18.1; no longer R18.2
- net N$34: no longer R18.1
- net N$40: now also R18.2
Routing:
- net N$40: track 27.7 -> 32.4 mm
- net PGND: track 83.1 -> 87.1 mm
- net N$34: track 12.8 -> 10.00 mm
- net N$29: track 11.6 -> 12.8 mm
Changed lines of the file:
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@@
 <wire x1="33.655" y1="45.72" x2="39.6875" y2="51.7525" width="0.8128" layer="21"/>
 <wire x1="39.6875" y1="51.7525" x2="39.6875" y2="63.97625" width="0.8128" layer="21"/>
+<wire x1="18.57375" y1="14.12875" x2="18.89125" y2="14.12875" width="0.2032" layer="42"/>
 </plain>
 <attributes>
@@
 <attribute name="VALUE" x="68.5675" y="10.53125" size="0.8128" layer="28" rot="MR180"/>
 </element>
-<element name="R17" library="my_rcl" package="1608" value="5k" x="59.69" y="7.77875" smashed="yes" rot="MR270">
+<element name="R17" library="my_rcl" package="1608" value="10k" x="59.69" y="7.77875" smashed="yes" rot="MR270">
 <attribute name="NAME" x="58.69" y="9.37875" size="0.8128" layer="26" rot="MR270"/>
 <attribute name="VALUE" x="58.725" y="10.53125" size="0.8128" layer="28" rot="MR180"/>
-</element>
-<element name="R18" library="my_rcl" package="1608" value="1.5k" x="59.69" y="3.96875" smashed="yes" rot="MR90">
-<attribute name="NAME" x="60.69" y="2.36875" size="0.8128" layer="26" rot="MR90"/>
-<attribute name="VALUE" x="57.7725" y="1.8" size="0.8128" layer="28" rot="MR180"/>
 </element>
 <element name="R19" library="my_rcl" package="1608" value="10k" x="61.9125" y="3.96875" smashed="yes" rot="MR270">
@@
 <attribute name="VALUE" x="10.795" y="27.305" size="0.8128" layer="28" rot="MR270"/>
 </element>
-<element name="R3" library="my_rcl" package="1608" value="" x="27.305" y="13.49375" smashed="yes" rot="MR90">
+<element name="R3" library="my_rcl" package="1608" value="10k" x="27.305" y="13.49375" smashed="yes" rot="MR90">
 <attribute name="NAME" x="28.305" y="11.89375" size="0.8128" layer="26" rot="MR90"/>
 <attribute name="VALUE" x="25.505" y="11.89375" size="0.8128" layer="28" rot="MR90"/>
@@
 <attribute name="VALUE" x="18.31" y="11.76" size="0.8128" layer="28" rot="MR270"/>
 </element>
-<element name="R9" library="my_rcl" package="1608" value="" x="19.685" y="13.49375" smashed="yes" rot="MR90">
+<element name="R9" library="my_rcl" package="1608" value="330" x="19.685" y="13.49375" smashed="yes" rot="MR90">
 <attribute name="NAME" x="20.685" y="11.89375" size="0.8128" layer="26" rot="MR90"/>
-<attribute name="VALUE" x="17.885" y="11.89375" size="0.8128" layer="28" rot="MR90"/>
-</element>
-<element name="C4" library="my_rcl" package="1608" value="" x="21.59" y="13.49375" smashed="yes" rot="MR270">
+<attribute name="VALUE" x="20.05625" y="11.60125" size="0.8128" layer="28" rot="MR270"/>
+</element>
+<element name="C4" library="my_rcl" package="1608" value="100p" x="21.59" y="13.49375" smashed="yes" rot="MR270">
 <attribute name="NAME" x="20.59" y="15.09375" size="0.8128" layer="26" rot="MR270"/>
-<attribute name="VALUE" x="23.39" y="15.09375" size="0.8128" layer="28" rot="MR270"/>
+<attribute name="VALUE" x="21.96125" y="11.60125" size="0.8128" layer="28" rot="MR270"/>
 </element>
 <element name="C5" library="my_rcl" package="1608" value="0.1u" x="25.0825" y="25.7175" smashed="yes" rot="MR0">
@@
 <attribute name="VALUE" x="22.8475" y="27.67625" size="0.8128" layer="28" rot="MR180"/>
 </element>
-<element name="C6" library="my_rcl" package="C050" value="1kV 470p" x="34.29" y="22.225" smashed="yes" rot="R270">
+<element name="C6" library="my_rcl" package="C050" value="1kV 22p" x="34.29" y="22.225" smashed="yes" rot="R270">
 <attribute name="NAME" x="36.195" y="25.781" size="0.8128" layer="25" ratio="10" rot="R270"/>
 <attribute name="VALUE" x="36.322" y="24.511" size="0.8128" layer="27" ratio="10" rot="R270"/>
@@
 <attribute name="NAME" x="63.07125" y="6.17875" size="0.8128" layer="26" rot="MR90"/>
 <attribute name="VALUE" x="61.10625" y="10.53125" size="0.8128" layer="28" rot="MR180"/>
+</element>
+<element name="R18" library="my_rcl" package="1608" value="10k" x="59.69" y="3.96875" smashed="yes" rot="MR90">
+<attribute name="NAME" x="60.69" y="2.36875" size="0.8128" layer="26" rot="MR90"/>
+<attribute name="VALUE" x="57.93125" y="1.8" size="0.8128" layer="28" rot="MR180"/>
 </element>
 </elements>
@@
 <wire x1="60.6425" y1="20.955" x2="55.88" y2="16.1925" width="1.27" layer="1"/>
 <via x="55.245" y="3.175" extent="1-16" drill="0.4"/>
-<via x="56.8325" y="5.715" extent="1-16" drill="0.4"/>
+<via x="57.4675" y="5.55625" extent="1-16" drill="0.4"/>
 <via x="58.26125" y="2.2225" extent="1-16" drill="0.4"/>
 <via x="67.31" y="1.11125" extent="1-16" drill="0.4"/>
 <via x="63.1825" y="2.2225" extent="1-16" drill="0.4"/>
 <via x="60.80125" y="7.77875" extent="1-16" drill="0.4"/>
-<via x="58.1025" y="7.77875" extent="1-16" drill="0.4"/>
+<via x="58.26125" y="8.89" extent="1-16" drill="0.4"/>
 <via x="63.65875" y="10.31875" extent="1-16" drill="0.4"/>
 <via x="71.4375" y="7.3025" extent="1-16" drill="0.4"/>
@@
 <contactref element="C11" pad="2"/>
 <wire x1="68.7125" y1="8.54625" x2="68.8975" y2="8.36125" width="0.2032" layer="16"/>
-<wire x1="59.69" y1="8.67875" x2="60.53625" y2="9.525" width="0.3048" layer="16"/>
-<wire x1="63.34125" y1="9.525" x2="60.53625" y2="9.525" width="0.3048" layer="16"/>
+<wire x1="60.53625" y1="9.525" x2="63.34125" y2="9.525" width="0.3048" layer="16"/>
 <wire x1="64.29375" y1="8.67875" x2="64.1875" y2="8.67875" width="0.3048" layer="16"/>
 <wire x1="64.1875" y1="8.67875" x2="63.34125" y2="9.525" width="0.3048" layer="16"/>
@@
 <wire x1="82.70875" y1="10.18125" x2="85.05875" y2="10.18125" width="0.3048" layer="16"/>
 <wire x1="85.05875" y1="10.18125" x2="85.09" y2="10.2125" width="0.3048" layer="16"/>
+<contactref element="R18" pad="2"/>
+<wire x1="59.69" y1="8.67875" x2="59.6375" y2="8.67875" width="0.3048" layer="16"/>
+<wire x1="58.7375" y1="5.82125" x2="59.69" y2="4.86875" width="0.3048" layer="16"/>
+<wire x1="59.6375" y1="8.67875" x2="58.7375" y2="7.77875" width="0.3048" layer="16"/>
+<wire x1="58.7375" y1="7.77875" x2="58.7375" y2="5.82125" width="0.3048" layer="16"/>
+<wire x1="59.69" y1="8.67875" x2="60.53625" y2="9.525" width="0.3048" layer="16"/>
 </signal>
 <signal name="N$6">
@@
 <contactref element="R19" pad="1"/>
 <contactref element="IC2" pad="3"/>
-<contactref element="R18" pad="2"/>
 <contactref element="Q3" pad="2"/>
-<wire x1="56.1975" y1="4.445" x2="59.26625" y2="4.445" width="0.2032" layer="16"/>
-<wire x1="59.26625" y1="4.445" x2="59.69" y2="4.86875" width="0.2032" layer="16"/>
-<wire x1="61.9125" y1="4.86875" x2="59.69" y2="4.86875" width="0.2032" layer="16"/>
 <wire x1="66.51625" y1="7.62" x2="64.77" y2="5.87375" width="0.2032" layer="16"/>
 <wire x1="62.9175" y1="5.87375" x2="61.9125" y2="4.86875" width="0.2032" layer="16"/>
 <wire x1="64.77" y1="5.87375" x2="62.9175" y2="5.87375" width="0.2032" layer="16"/>
+<contactref element="R18" pad="1"/>
+<wire x1="61.9125" y1="4.86875" x2="61.70125" y2="4.86875" width="0.2032" layer="16"/>
+<wire x1="59.90125" y1="3.06875" x2="59.69" y2="3.06875" width="0.2032" layer="16"/>
+<wire x1="61.70125" y1="4.86875" x2="59.90125" y2="3.06875" width="0.2032" layer="16"/>
+<wire x1="59.69" y1="3.06875" x2="59.6375" y2="3.01625" width="0.2032" layer="16"/>
+<wire x1="59.6375" y1="3.01625" x2="57.62625" y2="3.01625" width="0.2032" layer="16"/>
+<wire x1="57.62625" y1="3.01625" x2="56.1975" y2="4.445" width="0.2032" layer="16"/>
 </signal>
 <signal name="N$32">
@@
 <signal name="N$34">
 <contactref element="R17" pad="2"/>
-<contactref element="R18" pad="1"/>
 <contactref element="Q3" pad="1"/>
 <contactref element="R12" pad="1"/>
-<wire x1="56.1975" y1="1.905" x2="57.36125" y2="3.06875" width="0.2032" layer="16"/>
-<wire x1="57.36125" y1="3.06875" x2="59.69" y2="3.06875" width="0.2032" layer="16"/>
-<wire x1="58.52625" y1="5.715" x2="58.71125" y2="5.9" width="0.2032" layer="16"/>
-<wire x1="58.71125" y1="5.9" x2="59.69" y2="6.87875" width="0.2032" layer="16"/>
-<wire x1="59.69" y1="6.87875" x2="62.07125" y2="6.87875" width="0.2032" layer="16"/>
-<wire x1="56.1975" y1="1.905" x2="57.785" y2="3.4925" width="0.2032" layer="1"/>
-<wire x1="57.785" y1="3.4925" x2="57.785" y2="5.08" width="0.2032" layer="1"/>
-<via x="57.785" y="5.08" extent="1-16" drill="0.35"/>
-<wire x1="57.785" y1="5.08" x2="57.89125" y2="5.08" width="0.2032" layer="16"/>
-<wire x1="57.89125" y1="5.08" x2="58.52625" y2="5.715" width="0.2032" layer="16"/>
+<wire x1="59.69" y1="6.87875" x2="59.84875" y2="6.87875" width="0.2032" layer="16"/>
+<wire x1="59.84875" y1="6.87875" x2="62.07125" y2="6.87875" width="0.2032" layer="16"/>
+<wire x1="60.80125" y1="6.0325" x2="56.67375" y2="1.905" width="0.2032" layer="1"/>
+<wire x1="56.1975" y1="1.905" x2="56.67375" y2="1.905" width="0.2032" layer="1"/>
+<via x="60.80125" y="6.0325" extent="1-16" drill="0.35"/>
+<wire x1="60.80125" y1="6.0325" x2="60.695" y2="6.0325" width="0.2032" layer="16"/>
+<wire x1="60.695" y1="6.0325" x2="59.84875" y2="6.87875" width="0.2032" layer="16"/>
 </signal>
 <signal name="N$35">
@@
 <contactref element="C7" pad="2"/>
 <wire x1="20.32" y1="40.64" x2="20.32" y2="38.1" width="1.27" layer="16"/>
-<wire x1="20.32" y1="38.1" x2="20.32" y2="36.61125" width="1.27" layer="16"/>
-<wire x1="20.32" y1="36.61125" x2="18.63375" y2="34.925" width="1.27" layer="16"/>
+<wire x1="20.32" y1="36.61125" x2="20.32" y2="38.1" width="1.27" layer="16"/>
 <contactref element="C15" pad="2"/>
 <wire x1="30.32125" y1="32.22625" x2="34.29" y2="36.195" width="1.905" layer="1"/>
@@
 <via x="28.8925" y="12.54125" extent="1-16" drill="0.4"/>
 <via x="25.7175" y="16.03375" extent="1-16" drill="0.4"/>
+<wire x1="20.32" y1="40.64" x2="20.32" y2="36.61125" width="1.905" layer="16"/>
+<wire x1="20.32" y1="36.61125" x2="18.63375" y2="34.925" width="1.905" layer="16"/>
 </signal>
 <signal name="N$23">
