File: ac-adapter.brd (EAGLE design)
At the start: 87.6 x 73 mm, 67 parts, among them IC1 NCP13992, IC2 TL431, Q1 300V 5A, Q2 300V 5A, Q3 TLP621-1, Q4 BSS128, T1 COMMON_FILTER-SU10VFC, T2 TRANSFORMAER_FLYBACK-PQ2620

Commit message: tiny fix
Parts:
- added C12: 0.01u, my_rcl:1608
- added C13: 1kV 1000p, my_rcl:C050
- added R22: 1k, my_rcl:1608
- added R23: DNP, my_rcl:1608
- C23: device my_rcl:C100 -> my_rcl:C125
- C6: value 1kV 22p -> 1kV 1000p
- R6: value 10k -> 1k
- R7: value 10k -> 0; device my_rcl:1608 -> my_rcl:1608-J
- R9: value 330 -> 39
- moved R9 13.7 mm to (32.7, 17.8), turned to 180 degrees
- moved C6 2.29 mm to (35.6, 20.3)
- moved C4 1.91 mm to (19.7, 13.5)
- moved L3 1.60 mm to (53.8, 52.2)
- moved C23 1.27 mm to (34.3, 31.1)
Connections:
- new net N$27: C6.2, R22.2, R23.2, R9.2
- net N$14: now also R22.1; no longer C6.2, R9.2
- net N$19: now also C12.1
- net PGND: now also C12.2, C13.2, R23.1
- net SW: now also C13.1
Routing:
- net N$27: track 0.00 -> 18.9 mm, vias 0 -> 2
- net N$14: track 21.2 -> 5.47 mm, vias 1 -> 0
- net PGND: track 87.1 -> 97.0 mm, vias 51 -> 54
- net N$19: track 22.4 -> 24.3 mm
- net SW: track 55.3 -> 56.9 mm
- net N$8: track 10.2 -> 11.1 mm
- net N$11: track 6.32 -> 7.14 mm
Other:
- board text added: "LLC Power Supply v2.1"
- board text removed: "LLC Power Supply v2"
