File: ac-adapter.sch (EAGLE design)
At the start: 67 parts, among them IC1 NCP13992, IC2 TL431, Q1 300V 5A, Q2 300V 5A, Q3 TLP621-1, Q4 BSS128, T1 COMMON_FILTER-SU10VFC, T2 TRANSFORMAER_FLYBACK-PQ2620

Commit message: 微修正
Parts:
- C4: value (none) -> 100p
- C6: value 1kV 470p -> 1kV 22p
- R17: value 5k -> 10k
- R18: value 1.5k -> 10k
- R3: value (none) -> 10k
- R9: value (none) -> 330
Connections:
- net N$29: now also R18.1; no longer R18.2
- net N$34: no longer R18.1
- net N$40: now also R18.2
Other:
- moved on the sheet: C24, R12, R17, R18, R19

Commit message: tiny fix
Parts:
- added C12: 0.01u, my_rcl:C-1608
- added C13: 1kV 1000p, my_rcl:C-5
- added R22: 1k, my_rcl:R-1608
- added R23: DNP, my_rcl:R-1608
- C23: device my_rcl:C-10 -> my_rcl:C-12.5
- C6: value 1kV 22p -> 1kV 1000p
- R6: value 10k -> 1k
- R7: value 10k -> 0; device my_rcl:R-1608 -> my_rcl:R-1608J
- R9: value 330 -> 39
Connections:
- new net N$27: C6.2, R22.2, R23.2, R9.2
- net N$14: now also R22.1; no longer C6.2, R9.2
- net N$19: now also C12.1
- net PGND: now also C12.2, C13.2, R23.1
- net SW: now also C13.1
Other:
- moved on the sheet: C11, C15, C17, C18, C19, C20, C21, C22, C23, C24, C4, C6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
